Commit message: revised on old version

File: src/simulation/robots/a1_description/xacro/const.xacro (robot description, xacro)
@@ -90,5 +90,5 @@
     <!-- foot -->
     <xacro:property name="foot_mass" value="0.06"/>
-    <xacro:property name="foot_mu" value="0.8"/>
+    <xacro:property name="foot_mu" value="0.6"/>
     <xacro:property name="kp" value="100"/>
     <xacro:property name="kd" value="1"/>

File: src/simulation/robots/a1_description/xacro/gazebo.xacro (robot description, xacro)
@@ -40,10 +40,10 @@
         </plugin>
     </gazebo> -->
-   <!-- <gazebo>
-       <plugin filename="libgazebo_ros_force.so" name="gazebo_ros_force">
-           <bodyName>trunk</bodyName>
-           <topicName>/apply_force/trunk</topicName>
-       </plugin>
-    </gazebo> -->
+<!--    <gazebo>-->
+<!--        <plugin filename="libgazebo_ros_force.so" name="gazebo_ros_force">-->
+<!--            <bodyName>trunk</bodyName>-->
+<!--            <topicName>/apply_force/trunk</topicName>-->
+<!--        </plugin>-->
+<!--    </gazebo>-->
     <gazebo reference="imu_link">
         <gravity>true</gravity>
@@ -131,44 +131,4 @@
         </visual>
     </gazebo> -->
-    <!-- <gazebo>
-        <plugin filename="libnewLinkPlot3DPlugin.so" name="3dplot">
-            <frequency>1000</frequency>
-            <plot>
-                <link>FR_calf</link>
-                <pose>0 0 -0.2 0 0 0</pose>
-                <material>Gazebo/Yellow</material>
-            </plot>
-        </plugin>
-    </gazebo>
-    <gazebo>
-        <plugin filename="libnewLinkPlot3DPlugin.so" name="3dplot">
-            <frequency>1000</frequency>
-            <plot>
-                <link>FL_calf</link>
-                <pose>0 0 -0.2 0 0 0</pose>
-                <material>Gazebo/Red</material>
-            </plot>
-        </plugin>
-    </gazebo>
-    <gazebo>
-        <plugin filename="libnewLinkPlot3DPlugin.so" name="3dplot">
-            <frequency>1000</frequency>
-            <plot>
-                <link>RR_calf</link>
-                <pose>0 0 -0.2 0 0 0</pose>
-                <material>Gazebo/Blue</material>
-            </plot>
-        </plugin>
-    </gazebo>
-    <gazebo>
-        <plugin filename="libnewLinkPlot3DPlugin.so" name="3dplot">
-            <frequency>1000</frequency>
-            <plot>
-                <link>RL_calf</link>
-                <pose>0 0 -0.2 0 0 0</pose>
-                <material>Gazebo/Black</material>
-            </plot>
-        </plugin>
-    </gazebo> -->
     <!-- Show planned pose location -->
      <!-- <gazebo reference="base">
@@ -179,14 +139,4 @@
         </visual>
     </gazebo> -->
-    <!-- <gazebo>
-        <plugin filename="libLinkPlot3DPlugin.so" name="3dplotTrunk">
-            <frequency>10</frequency>
-            <plot>
-                <link>base</link>
-                <pose>0 0 0 0 0 0</pose>
-                <material>Gazebo/Yellow</material>
-            </plot>
-        </plugin>
-  </gazebo> -->
     <gazebo reference="base">
         <material>Gazebo/Green</material>
