Commit message: add factory function and mpc demo

File: simulation/robots/a1_description/xacro/leg.xacro (robot description, xacro)
@@ -73,5 +73,5 @@
             <dynamics damping="${damping}" friction="${friction}"/>
             <limit effort="${thigh_torque_max}" velocity="${thigh_velocity_max}" lower="${thigh_min*PI/180.0}" upper="${thigh_max*PI/180.0}"/>
-        </joint>
+        </joint>r
         <link name="${name}_thigh">
             <visual>
