Commit message: Add the sensor of a1

File: simulation/robots/a1_description/xacro/robot.xacro (robot description, xacro)
@@ -7,5 +7,11 @@
     <xacro:include filename="$(find a1_description)/xacro/gazebo.xacro"/>
     <xacro:if value="$(arg USE_CAMERA)">
-        <xacro:include filename="$(find realsense_ros_gazebo)/xacro/depthcam.xacro"/>
+        <xacro:include filename="$(find a1_description)/xacro/realsense_d435.xacro"/>
+    </xacro:if>
+    <xacro:if value="$(arg USE_LASER)">
+        <xacro:include filename="$(find a1_description)/xacro/VLP-16.xacro"/>
+    </xacro:if>
+    <xacro:if value="$(arg USE_GPS)">
+        <xacro:include filename="$(find a1_description)/xacro/gps_gazebo.xacro"/>
     </xacro:if>
     <!-- <xacro:include filename="$(find a1_gazebo)/launch/stairs.urdf.xacro"/> -->
@@ -64,8 +70,122 @@
         </inertial>
     </link>
+    <link name="fulcrum1">
+         <visual>
+             <origin xyz="0 0 0" rpy="0 0 0" />
+             <geometry>
+                <box size="0 0 0"/>
+            </geometry>
+            <material name="orange"/>
+        </visual>
+        <collision>
+              <origin rpy="0 0 0" xyz="0 0 0"/>
+           <geometry>
+                <box size="0.01 0.01 0.13"/>
+          </geometry>
+        </collision>
+    </link>
+    <joint name="fulcrum1_joint" type="fixed">
+            <origin xyz="0.12 0.09 0" rpy="0 0 0"/>
+            <parent link="trunk"/>
+            <child link="fulcrum1"/>
+    </joint>
+    <link name="fulcrum2">
+         <visual>
+             <origin xyz="0 0 0" rpy="0 0 0" />
+             <geometry>
+                <box size="0 0 0"/>
+            </geometry>
+            <material name="orange"/>
+        </visual>
+        <collision>
+              <origin rpy="0 0 0" xyz="0 0 0"/>
+           <geometry>
+                <box size="0.01 0.01 0.13"/>
+          </geometry>
+        </collision>
+    </link>
+    <joint name="fulcrum2_joint" type="fixed">
+            <origin xyz="-0.12 0.09 0" rpy="0 0 0"/>
+            <parent link="trunk"/>
+            <child link="fulcrum2"/>
+    </joint>
+        <link name="fulcrum3">
+         <visual>
+             <origin xyz="0 0 0" rpy="0 0 0" />
+             <geometry>
+                <box size="0 0 0"/>
+            </geometry>
+            <material name="orange"/>
+        </visual>
+        <collision>
+              <origin rpy="0 0 0" xyz="0 0 0"/>
+           <geometry>
+                <box size="0.01 0.01 0.13"/>
+          </geometry>
+        </collision>
+    </link>
+    <joint name="fulcrum3_joint" type="fixed">
+            <origin xyz="0.12 -0.09 0" rpy="0 0 0"/>
+            <parent link="trunk"/>
+            <child link="fulcrum3"/>
+    </joint>
+        <link name="fulcrum4">
+         <visual>
+             <origin xyz="0 0 0" rpy="0 0 0" />
+             <geometry>
+                <box size="0 0 0"/>
+            </geometry>
+            <material name="orange"/>
+        </visual>
+        <collision>
+              <origin rpy="0 0 0" xyz="0 0 0"/>
+           <geometry>
+                <box size="0.01 0.01 0.13"/>
+          </geometry>
+        </collision>
+    </link>
+    <joint name="fulcrum4_joint" type="fixed">
+            <origin xyz="-0.12 -0.09 0" rpy="0 0 0"/>
+            <parent link="trunk"/>
+            <child link="fulcrum4"/>
+    </joint>
     <xacro:if value="$(arg USE_CAMERA)">
         <xacro:realsense_d435 sensor_name="d435" parent_link="trunk" rate="10">
             <origin rpy="0 0 0 " xyz="0.25 0 0.055"/>
         </xacro:realsense_d435>
+    </xacro:if>
+    <xacro:if value="$(arg USE_LASER)">
+        <xacro:VLP-16 sensor_name="velodyne" parent= "trunk" rate= "15">
+            <origin rpy="0 0 0 " xyz="0 0 0.055"/>
+        </xacro:VLP-16>
+    </xacro:if>
+    <xacro:if value="$(arg USE_GPS)">
+         <joint name="gps_joint" type="fixed">
+                <parent link="trunk"/>
+                <child link="gps_link"/>
+         </joint>
+        <link name="gps_link">
+            <collision>
+            <origin xyz="0 0 0" rpy="0 0 0"/>
+            <geometry>
+                <box size="0.01 0.01 0.01"/>
+            </geometry>
+            </collision>
+            <visual>
+            <origin xyz="0 0 0" rpy="0 0 0"/>
+            <geometry>
+                <box size="0.01 0.01 0.01"/>
+            </geometry>
+            <material name="orange"/>
+            </visual>
+            <inertial>
+            <origin xyz="0 0 0" rpy="0 0 0"/>
+            <mass value="0.01"/>
+            <inertia
+                ixx="1.0" ixy="0.0" ixz="0.0"
+                iyy="1.0" iyz="0.0"
+                izz="1.0"/>
+            </inertial>
+        </link>
     </xacro:if>
     <xacro:if value="${(rolloverProtection == 'true')}">

Commit message: Remove the excess link of a1_xacro

File: simulation/robots/a1_description/xacro/robot.xacro (robot description, xacro)
@@ -70,84 +70,4 @@
         </inertial>
     </link>
-    <link name="fulcrum1">
-         <visual>
-             <origin xyz="0 0 0" rpy="0 0 0" />
-             <geometry>
-                <box size="0 0 0"/>
-            </geometry>
-            <material name="orange"/>
-        </visual>
-        <collision>
-              <origin rpy="0 0 0" xyz="0 0 0"/>
-           <geometry>
-                <box size="0.01 0.01 0.13"/>
-          </geometry>
-        </collision>
-    </link>
-    <joint name="fulcrum1_joint" type="fixed">
-            <origin xyz="0.12 0.09 0" rpy="0 0 0"/>
-            <parent link="trunk"/>
-            <child link="fulcrum1"/>
-    </joint>
-    <link name="fulcrum2">
-         <visual>
-             <origin xyz="0 0 0" rpy="0 0 0" />
-             <geometry>
-                <box size="0 0 0"/>
-            </geometry>
-            <material name="orange"/>
-        </visual>
-        <collision>
-              <origin rpy="0 0 0" xyz="0 0 0"/>
-           <geometry>
-                <box size="0.01 0.01 0.13"/>
-          </geometry>
-        </collision>
-    </link>
-    <joint name="fulcrum2_joint" type="fixed">
-            <origin xyz="-0.12 0.09 0" rpy="0 0 0"/>
-            <parent link="trunk"/>
-            <child link="fulcrum2"/>
-    </joint>
-        <link name="fulcrum3">
-         <visual>
-             <origin xyz="0 0 0" rpy="0 0 0" />
-             <geometry>
-                <box size="0 0 0"/>
-            </geometry>
-            <material name="orange"/>
-        </visual>
-        <collision>
-              <origin rpy="0 0 0" xyz="0 0 0"/>
-           <geometry>
-                <box size="0.01 0.01 0.13"/>
-          </geometry>
-        </collision>
-    </link>
-    <joint name="fulcrum3_joint" type="fixed">
-            <origin xyz="0.12 -0.09 0" rpy="0 0 0"/>
-            <parent link="trunk"/>
-            <child link="fulcrum3"/>
-    </joint>
-        <link name="fulcrum4">
-         <visual>
-             <origin xyz="0 0 0" rpy="0 0 0" />
-             <geometry>
-                <box size="0 0 0"/>
-            </geometry>
-            <material name="orange"/>
-        </visual>
-        <collision>
-              <origin rpy="0 0 0" xyz="0 0 0"/>
-           <geometry>
-                <box size="0.01 0.01 0.13"/>
-          </geometry>
-        </collision>
-    </link>
-    <joint name="fulcrum4_joint" type="fixed">
-            <origin xyz="-0.12 -0.09 0" rpy="0 0 0"/>
-            <parent link="trunk"/>
-            <child link="fulcrum4"/>
-    </joint>
     <xacro:if value="$(arg USE_CAMERA)">
         <xacro:realsense_d435 sensor_name="d435" parent_link="trunk" rate="10">
