Commit message: Modify the parameter of lidar,unify the control

File: simulation/robots/a1_description/xacro/VLP-16.xacro (robot description, xacro)
@@ -5,11 +5,11 @@
     <xacro:property name="topic" value="/velodyne_points"/>
     <xacro:property name="lasers" value="16"/>
-    <xacro:property name="samples" value="1875"/>
+    <xacro:property name="samples" value="1024"/>
     <xacro:property name="collision_range" value="0.3"/>
     <xacro:property name="min_range" value="0.9"/>
-    <xacro:property name="max_range" value="130.0"/>
+    <xacro:property name="max_range" value="100"/>
     <xacro:property name="min_angle" value="-${M_PI} "/>
     <xacro:property name="max_angle" value="${M_PI} "/>
-    <xacro:property name="gpu" value="true"/>
+    <xacro:property name="gpu" value="false"/>
     <xacro:property name="noise" value="0.008"/>
     <joint name="${sensor_name}_base_mount_joint" type="fixed">

File: simulation/robots/a1_description/xacro/robot.xacro (robot description, xacro)
@@ -76,5 +76,5 @@
     </xacro:if>
     <xacro:if value="$(arg USE_LIDAR)">
-        <xacro:VLP-16 sensor_name="velodyne" parent= "trunk" rate= "15">
+        <xacro:VLP-16 sensor_name="velodyne" parent= "trunk" rate= "10">
             <origin rpy="0 0 0 " xyz="0 0 0.055"/>
         </xacro:VLP-16>

Commit message: Improve some params

File: simulation/robots/a1_description/xacro/VLP-16.xacro (robot description, xacro)
@@ -5,11 +5,11 @@
     <xacro:property name="topic" value="/velodyne_points"/>
     <xacro:property name="lasers" value="16"/>
-    <xacro:property name="samples" value="1875"/>
+    <xacro:property name="samples" value="1024"/>
     <xacro:property name="collision_range" value="0.3"/>
     <xacro:property name="min_range" value="0.9"/>
-    <xacro:property name="max_range" value="130.0"/>
+    <xacro:property name="max_range" value="100.0"/>
     <xacro:property name="min_angle" value="-${M_PI} "/>
     <xacro:property name="max_angle" value="${M_PI} "/>
-    <xacro:property name="gpu" value="true"/>
+    <xacro:property name="gpu" value="false"/>
     <xacro:property name="noise" value="0.008"/>
     <joint name="${sensor_name}_base_mount_joint" type="fixed">
