Commit message: add lite2

File: simulation/robots/lite2_description/urdf/robot.urdf (robot description, URDF)
Before this commit: robot lite2_description, 14 links, 13 joints
Links:
- added link FL_FOOT, mass 1E-12; collision sphere radius=0.024
- added link FR_FOOT, mass 1E-12; collision sphere radius=0.024
- added link HL_FOOT, mass 1E-12; collision sphere radius=0.024
- added link HR_FOOT, mass 1E-12; collision sphere radius=0.024
- link FL_SHANK: geometry collision box size=0.02 0.02 0.16; visual mesh filename=package://lite2_description/meshes/SHANK.dae
- link FL_THIGH: geometry collision box size=0.03 0.03 0.16; visual mesh filename=package://lite2_description/meshes/L_THIGH.dae
- link FR_SHANK: geometry collision box size=0.02 0.02 0.16; visual mesh filename=package://lite2_description/meshes/SHANK.dae
- link FR_THIGH: geometry collision box size=0.03 0.03 0.16; visual mesh filename=package://lite2_description/meshes/R_THIGH2.dae
- link HL_SHANK: geometry collision box size=0.02 0.02 0.16; visual mesh filename=package://lite2_description/meshes/SHANK.dae
- link HL_THIGH: geometry collision box size=0.03 0.03 0.16; visual mesh filename=package://lite2_description/meshes/L_THIGH.dae
- link HR_SHANK: geometry collision box size=0.02 0.02 0.16; visual mesh filename=package://lite2_description/meshes/SHANK.dae
- link HR_THIGH: geometry collision box size=0.03 0.03 0.16; visual mesh filename=package://lite2_description/meshes/R_THIGH2.dae
- link TORSO: geometry collision box size=0.234 0.184 0.08; visual mesh filename=package://lite2_description/meshes/TORSO2.dae
Joints:
- removed joint FL_HipX
- removed joint FL_HipY
- removed joint FL_Knee
- removed joint FR_HipX
- removed joint FR_HipY
- removed joint FR_Knee
- removed joint HL_HipX
- removed joint HL_HipY
- removed joint HL_Knee
- removed joint HR_HipX
- removed joint HR_HipY
- removed joint HR_Knee
- added joint FL_calf_joint: type revolute, parent FL_THIGH, child FL_SHANK, origin xyz=0 0 -0.18 rpy=0 0 0, axis 0 -1 0, limit lower=0.419 upper=2.53 effort=28 velocity=20
- added joint FL_foot_fixed: type fixed, parent FL_SHANK, child FL_FOOT, origin xyz=0 0 -0.19 rpy=0 0 0
- added joint FL_hip_joint: type revolute, parent TORSO, child FL_HIP, origin xyz=0.175 0.055 0 rpy=0 0 0, axis 1 0 0, limit lower=-0.523 upper=0.523 effort=13.2 velocity=20
- added joint FL_thigh_joint: type revolute, parent FL_HIP, child FL_THIGH, origin xyz=0 0.081 0 rpy=0 0 0, axis 0 -1 0, limit lower=-3.49 upper=0.349 effort=13.2 velocity=20
- added joint FR_calf_joint: type revolute, parent FR_THIGH, child FR_SHANK, origin xyz=0 0 -0.18 rpy=0 0 0, axis 0 -1 0, limit lower=0.419 upper=2.53 effort=28 velocity=20
- added joint FR_foot_fixed: type fixed, parent FR_SHANK, child FR_FOOT, origin xyz=0 0 -0.19 rpy=0 0 0
- added joint FR_hip_joint: type revolute, parent TORSO, child FR_HIP, origin xyz=0.175 -0.055 0 rpy=0 0 0, axis -1 0 0, limit lower=-0.523 upper=0.523 effort=13.2 velocity=20
- added joint FR_thigh_joint: type revolute, parent FR_HIP, child FR_THIGH, origin xyz=0 -0.08 0 rpy=0 0 0, axis 0 -1 0, limit lower=-3.49 upper=0.349 effort=13.2 velocity=20
- added joint RL_calf_joint: type revolute, parent HL_THIGH, child HL_SHANK, origin xyz=0 0 -0.18 rpy=0 0 0, axis 0 -1 0, limit lower=0.419 upper=2.53 effort=28 velocity=20
- added joint RL_foot_fixed: type fixed, parent HL_SHANK, child HL_FOOT, origin xyz=0 0 -0.19 rpy=0 0 0
- added joint RL_hip_joint: type revolute, parent TORSO, child HL_HIP, origin xyz=-0.175 0.055 0 rpy=0 0 0, axis 1 0 0, limit lower=-0.523 upper=0.523 effort=13.2 velocity=20
- added joint RL_thigh_joint: type revolute, parent HL_HIP, child HL_THIGH, origin xyz=0 0.081 0 rpy=0 0 0, axis 0 -1 0, limit lower=-3.49 upper=0.349 effort=13.2 velocity=20
- added joint RR_calf_joint: type revolute, parent HR_THIGH, child HR_SHANK, origin xyz=0 0 -0.18 rpy=0 0 0, axis 0 -1 0, limit lower=0.419 upper=2.53 effort=28 velocity=20
- added joint RR_foot_fixed: type fixed, parent HR_SHANK, child HR_FOOT, origin xyz=0 0 -0.19 rpy=0 0 0
- added joint RR_hip_joint: type revolute, parent TORSO, child HR_HIP, origin xyz=-0.175 -0.055 0 rpy=0 0 0, axis -1 0 0, limit lower=-0.523 upper=0.523 effort=13.2 velocity=20
- added joint RR_thigh_joint: type revolute, parent HR_HIP, child HR_THIGH, origin xyz=0 -0.081 0 rpy=0 0 0, axis 0 -1 0, limit lower=-3.49 upper=0.349 effort=13.2 velocity=20

Commit message: add imu plguin to lite2 urdf and fix some license for .h

File: simulation/robots/lite2_description/urdf/robot.urdf (robot description, URDF)
Before this commit: robot MiniLiteV2, 18 links, 17 joints
Links:
- added link imu_link, mass 0.001; collision box size=.001 .001 .001; visual box size=0.001 0.001 0.001
Joints:
- added joint imu_joint: type fixed, parent TORSO, child imu_link, origin xyz=0 0 0 rpy=0 0 0

Commit message: add simulation of Lite2

File: simulation/robots/lite2_description/urdf/robot.urdf (robot description, URDF)
Before this commit: robot MiniLiteV2, 19 links, 18 joints
Joints:
- removed joint FL_calf_joint
- removed joint FR_calf_joint
- removed joint RL_calf_joint
- removed joint RL_foot_fixed
- removed joint RL_hip_joint
- removed joint RL_thigh_joint
- removed joint RR_calf_joint
- removed joint RR_foot_fixed
- removed joint RR_hip_joint
- removed joint RR_thigh_joint
- added joint FL_shank_joint: type revolute, parent FL_THIGH, child FL_SHANK, origin xyz=0 0 -0.18 rpy=0 0 0, axis 0 1 0, limit lower=-2.53 upper=-0.419 effort=28 velocity=20
- added joint FR_shank_joint: type revolute, parent FR_THIGH, child FR_SHANK, origin xyz=0 0 -0.18 rpy=0 0 0, axis 0 1 0, limit lower=-2.53 upper=-0.419 effort=28 velocity=20
- added joint HL_foot_fixed: type fixed, parent HL_SHANK, child HL_FOOT, origin xyz=0 0 -0.19 rpy=0 0 0
- added joint HL_hip_joint: type revolute, parent TORSO, child HL_HIP, origin xyz=-0.175 0.055 0 rpy=0 0 0, axis 1 0 0, limit lower=-0.523 upper=0.523 effort=13.2 velocity=20
- added joint HL_shank_joint: type revolute, parent HL_THIGH, child HL_SHANK, origin xyz=0 0 -0.18 rpy=0 0 0, axis 0 1 0, limit lower=-2.53 upper=-0.419 effort=28 velocity=20
- added joint HL_thigh_joint: type revolute, parent HL_HIP, child HL_THIGH, origin xyz=0 0.081 0 rpy=0 0 0, axis 0 1 0, limit lower=-0.349 upper=3.49 effort=13.2 velocity=20
- added joint HR_foot_fixed: type fixed, parent HR_SHANK, child HR_FOOT, origin xyz=0 0 -0.19 rpy=0 0 0
- added joint HR_hip_joint: type revolute, parent TORSO, child HR_HIP, origin xyz=-0.175 -0.055 0 rpy=0 0 0, axis 1 0 0, limit lower=-0.523 upper=0.523 effort=13.2 velocity=20
- added joint HR_shank_joint: type revolute, parent HR_THIGH, child HR_SHANK, origin xyz=0 0 -0.18 rpy=0 0 0, axis 0 1 0, limit lower=-2.53 upper=-0.419 effort=28 velocity=20
- added joint HR_thigh_joint: type revolute, parent HR_HIP, child HR_THIGH, origin xyz=0 -0.081 0 rpy=0 0 0, axis 0 1 0, limit lower=-0.349 upper=3.49 effort=13.2 velocity=20
- joint FL_thigh_joint: axis 0 -1 0 -> 0 1 0; limit lower=-3.49 upper=0.349 effort=13.2 velocity=20 -> lower=-0.349 upper=3.49 effort=13.2 velocity=20
- joint FR_hip_joint: axis -1 0 0 -> 1 0 0
- joint FR_thigh_joint: axis 0 -1 0 -> 0 1 0; limit lower=-3.49 upper=0.349 effort=13.2 velocity=20 -> lower=-0.349 upper=3.49 effort=13.2 velocity=20
