Commit message: change SHANK.dae for lite3

File: robot_description/lite3_description/xacro/body.xacro (robot description, xacro)
@@ -79,5 +79,4 @@
       </inertial>
       <visual>
-        <origin rpy="0.88 0 1.5708" xyz="-0.171 0.25 -0.274"/>
         <geometry>
           <mesh filename="package://lite3_description/meshes/SHANK.dae" />
@@ -167,5 +166,4 @@
       </inertial>
       <visual>
-        <origin rpy="0.88 0 1.5708" xyz="-0.171 0.25 -0.274"/>
         <geometry>
           <mesh filename="package://lite3_description/meshes/SHANK.dae" />
@@ -255,5 +253,4 @@
       </inertial>
       <visual>
-        <origin rpy="0.88 0 1.5708" xyz="-0.171 0.25 -0.274"/>
         <geometry>
           <mesh filename="package://lite3_description/meshes/SHANK.dae" />
@@ -343,5 +340,4 @@
       </inertial>
       <visual>
-        <origin rpy="0.88 0 1.5708" xyz="-0.171 0.25 -0.274"/>
         <geometry>
           <mesh filename="package://lite3_description/meshes/SHANK.dae" />

Commit message: currently trot right

File: robot_description/lite3_description/xacro/body.xacro (robot description, xacro)
@@ -109,5 +109,5 @@
     </link>
     <joint name="FL_Ankle" type="fixed">
-      <origin xyz="0 0 -0.21"/>
+      <origin xyz="0 0 -0.20"/>
       <parent link="FL_SHANK" />
       <child link="FL_FOOT" />
@@ -196,5 +196,5 @@
     </link>
     <joint name="FR_Ankle" type="fixed">
-      <origin xyz="0 0 -0.21"/>
+      <origin xyz="0 0 -0.20"/>
       <parent link="FR_SHANK" />
       <child link="FR_FOOT" />
@@ -283,5 +283,5 @@
     </link>
     <joint name="HL_Ankle" type="fixed">
-      <origin xyz="0 0 -0.21"/>
+      <origin xyz="0 0 -0.20"/>
       <parent link="HL_SHANK" />
       <child link="HL_FOOT" />
@@ -370,5 +370,5 @@
     </link>
     <joint name="HR_Ankle" type="fixed">
-      <origin xyz="0 0 -0.21"/>
+      <origin xyz="0 0 -0.20"/>
       <parent link="HR_SHANK" />
       <child link="HR_FOOT" />
